File: cascade_cart_rev0/cascade_cart_rev0.kicad_pcb (KiCad board)
At the start: 2 copper layers, 88.9 x 129.5 mm, 26 parts, among them J1 Screw_Terminal_01x02, J2 Conn_01x03_Pin, J3 Conn_02x08_Counter_Clockwise, J4 Conn_01x02_Pin, J5 Conn_01x02_Pin, J6 Conn_01x06_Pin, J7 Conn_01x01_Pin, SW1 SW_SPDT

Commit message: update pcb
Other:
- board text added: "+3.3V"
- board text added: "GPIO34"
- board text added: "GPIO36"
- board text added: "VUSB"
- board text removed: "GPIO11"
Changed lines of the file:
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@@
     (property "Sheetname" "")
     (attr through_hole)
-    (fp_text reference "U1" (at 11.43 -5.08 90 unlocked) (layer "F.SilkS")
+    (fp_text reference "U1" (at 11.43 -16.51 unlocked) (layer "F.SilkS")
         (effects (font (size 1 1) (thickness 0.1)))
     )
@@
     (effects (font (size 1 1) (thickness 0.15)) (justify left bottom))
   )
-  (gr_text "ESP32-S2-Mini" (at 128.27 86.36) (layer "F.SilkS")
+  (gr_text "ESP32-S2-Mini" (at 125.73 73.66) (layer "F.SilkS")
     (effects (font (size 1 1) (thickness 0.15)) (justify left bottom))
   )
@@
     (effects (font (size 1 1) (thickness 0.15)) (justify left bottom))
   )
-  (gr_text "1N4001\n" (at 147.32 57.15 90) (layer "F.SilkS")
+  (gr_text "1N4001\n" (at 149.86 57.15 90) (layer "F.SilkS")
     (effects (font (size 1 1) (thickness 0.15)) (justify left bottom))
   )
@@
     (effects (font (size 1 1) (thickness 0.15)) (justify left bottom))
   )
-  (gr_text "GPIO11" (at 78.74 71.12) (layer "F.SilkS")
+  (gr_text "GPIO34" (at 74.93 88.9) (layer "F.SilkS")
+    (effects (font (size 1 1) (thickness 0.15)) (justify left bottom))
+  )
+  (gr_text "GND" (at 114.3 119.38) (layer "F.SilkS")
+    (effects (font (size 1 1) (thickness 0.15)) (justify left bottom))
+  )
+  (gr_text "GPIO36" (at 78.74 71.12) (layer "F.SilkS")
     (effects (font (size 1 1) (thickness 0.15)) (justify left bottom))
   )
@@
     (effects (font (size 1 1) (thickness 0.15)) (justify left bottom))
   )
+  (gr_text "GND\n" (at 96.52 119.38) (layer "F.SilkS")
+    (effects (font (size 1 1) (thickness 0.15)) (justify left bottom))
+  )
   (gr_text "GND\n" (at 119.38 100.33) (layer "F.SilkS")
     (effects (font (size 1 1) (thickness 0.15)) (justify left bottom))
@@
     (effects (font (size 1 1) (thickness 0.15)) (justify left bottom))
   )
+  (gr_text "+3.3V\n" (at 140.97 91.44) (layer "F.SilkS")
+    (effects (font (size 1 1) (thickness 0.15)) (justify left bottom))
+  )
   (gr_text "B2" (at 119.38 105.41) (layer "F.SilkS")
     (effects (font (size 1 1) (thickness 0.15)) (justify left bottom))
   )
+  (gr_text "VUSB\n" (at 147.32 57.15 90) (layer "F.SilkS")
+    (effects (font (size 1 1) (thickness 0.15)) (justify left bottom))
+  )

Commit message: prod files
Parts:
- added C1: 0.1uf, Capacitor_THT:C_Disc_D4.3mm_W1.9mm_P5.00mm, F.Cu at (115.6, 88.3)
- added C2: 0.1uf, Capacitor_THT:C_Disc_D4.3mm_W1.9mm_P5.00mm, F.Cu at (107.9, 114.9)
- added C3: 0.1uf, Capacitor_THT:C_Disc_D4.3mm_W1.9mm_P5.00mm, F.Cu at (141.0, 55.9)
- moved D1 4.58 mm to (141.0, 52.1), turned to 0 degrees
Routing:
- net +5V: track 186.7 -> 181.4 mm
- net /VUSB: track 3.81 -> 8.67 mm
- net /MOT_CONT_B1: track 25.6 -> 27.1 mm
- net /EN_A: track 28.2 -> 27.1 mm
