File: cascade_cart_rev0/cascade_cart_rev0.kicad_sch (KiCad schematic)
At the start: 26 parts, among them J1 Screw_Terminal_01x02, J2 Conn_01x03_Pin, J3 Conn_02x08_Counter_Clockwise, J4 Conn_01x02_Pin, J5 Conn_01x02_Pin, J6 Conn_01x06_Pin, J7 Conn_01x01_Pin, SW1 SW_SPDT

Commit message: prod files
Parts:
- added C1, C2, C3: 0.1uf, Capacitor_THT:C_Disc_D4.3mm_W1.9mm_P5.00mm, symbol Device:C
Connections:
- net +5V: now also C1.1, C2.1
- net GND: now also C1.2, C2.2, C3.2
- net VUSB: now also C3.1
Other:
- moved on the sheet: H1, H2, H3, H4, H5, H6, H7, H8, H9, J2, J7
